File: mouse_v2.sch (KiCad schematic (older format))
At the start: 74 parts, among them J1 HC05 Header, J2 Serial Debug Header, J3 HC05_Key Jump, M1 Conn_01x06_Female, M2 Conn_01x06_Female, Q0 Q_Photo_NPN, Q1 Q_Photo_NPN, Q2 Q_Photo_NPN, Q3 Q_Photo_NPN, T0 Q_NMOS_DGS, T1 Q_NMOS_DGS, T2 Q_NMOS_DGS, T3 Q_NMOS_DGS, T4 Q_NMOS_DGS, U2 L293D, U3 LM1085-5.0

Commit message: more shcem updates
Parts:
- removed T0, T1, T2, T3: Q_NMOS_DGS, misc:TN0104(TO-92)v2, symbol mouse_v2-rescue:Q_NMOS_DGS-Device
- added C5, C6, C7, C8: 22pF, symbol Device:C_Small
- added FB1, FB2, FB3, FB4: HZ0603C601R-10, symbol Device:FerriteBead_Small
- added J?: Conn_01x05_Male, symbol Connector:Conn_01x05_Male
- added Q4, Q5, Q6, Q7: Q_NMOS_SGD, symbol Device:Q_NMOS_SGD
- added R11: 10K, symbol Device:R
- TP1: value TestPoint -> V_EXT_TP
- TP2: value GND TP -> GND_TP
- gave numbers to parts that had none: 6
Connections:
- wire segments 238 -> 283
Other:
- note added: "* Select voltage divider resistors such\n that voltage at V_METER will not exceed\n the voltage limit on a pin"
- note removed: "*"
- moved on the sheet: BT_MH1, BT_MH2, D4, D5, D6, ERM1_1, ERM1_2, ERM1_3, ERM1_4, ERM2_1, ERM2_2, ERM2_3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

Commit message: s
Parts:
- added JP2: JP_GND, Jumper:SolderJumper-2_P1.3mm_Open_Pad1.0x1.5mm, symbol Jumper:SolderJumper_2_Open
- added JP3: JP_RST, Jumper:SolderJumper-2_P1.3mm_Open_Pad1.0x1.5mm, symbol Jumper:SolderJumper_2_Open
- added Q8: Q_NMOS_SGD, Package_TO_SOT_THT:TO-92, symbol Device:Q_NMOS_SGD
- C1, C2: footprint (none) -> Capacitor_THT:CP_Radial_D6.3mm_P2.50mm
- C3, C4: footprint (none) -> Capacitor_SMD:C_1206_3216Metric_Pad1.33x1.80mm_HandSolder
- C5, C6, C7, C8: footprint (none) -> Capacitor_SMD:C_0603_1608Metric_Pad1.08x0.95mm_HandSolder
- D4, D5, D6: footprint LED_SMD:LED_0201_0603Metric_Pad0.64x0.40mm_HandSolder -> LED_SMD:LED_0805_2012Metric_Pad1.15x1.40mm_HandSolder
- FB1, FB2, FB3, FB4: footprint (none) -> Resistor_SMD:R_0603_1608Metric_Pad0.98x0.95mm_HandSolder
- J4: footprint (none) -> Connector_PinHeader_1.27mm:PinHeader_2x05_P1.27mm_Vertical
- J5: renamed from J?; value Conn_01x05_Male -> SWD Header; footprint (none) -> Connector_PinHeader_2.54mm:PinHeader_1x05_P2.54mm_Vertical
- JP1: value Jumper -> JP_SWO; footprint (none) -> Jumper:SolderJumper-2_P1.3mm_Open_Pad1.0x1.5mm
- M1: value Conn_01x06_Female -> M1_Conn; footprint (none) -> Connector_PinHeader_1.00mm:PinHeader_1x06_P1.00mm_Vertical
- M2: value Conn_01x06_Female -> M2_Conn; footprint (none) -> Connector_PinHeader_1.00mm:PinHeader_1x06_P1.00mm_Vertical
- Q4, Q5, Q6, Q7: footprint (none) -> Package_TO_SOT_THT:TO-92
- R1, R13, R14, R15, R16, R17, R18, R2, R22, R23, R3, R4, R5, R6, R7, R8: footprint Resistor_THT:R_Axial_DIN0207_L6.3mm_D2.5mm_P10.16mm_Horizontal -> Resistor_SMD:R_1206_3216Metric_Pad1.30x1.75mm_HandSolder
- R10, R11, R9: footprint (none) -> Resistor_SMD:R_1206_3216Metric_Pad1.30x1.75mm_HandSolder
- S1: footprint misc:SWITCH_SLIDE_500SSP1S2M2QEA -> custom:1103M2S4CQE2
- SW1: footprint (none) -> Button_Switch_THT:SW_PUSH_6mm
- T4: footprint misc:TN0104(TO-92)v2 -> Package_TO_SOT_THT:TO-92
- TP1, TP2: footprint (none) -> Connector_PinHeader_2.54mm:PinHeader_1x01_P2.54mm_Vertical
- U1: footprint (none) -> bluepill:YAAJ_BluePill_SWD_2
Connections:
- wire segments 283 -> 290

Commit message: wip
Parts:
- removed ERM1_1, ERM1_2, ERM1_3, ERM1_4, ERM2_1, ERM2_2, ERM2_3, ERM2_4: M2, MountingHole:MountingHole_2.2mm_M2, symbol mouse_v2-rescue:MountingHole-Mechanical
- removed T4: Q_NMOS_DGS, Package_TO_SOT_THT:TO-92, symbol mouse_v2-rescue:Q_NMOS_DGS-Device
- added MH1: M1_MH, custom:Motor_mouse, symbol Motor:Motor_DC
- added MH2: M2_MH, custom:Motor_mouse, symbol Motor:Motor_DC
- added S2: EG1218, custom:1103M2S4CQE2, symbol mouse-rescue:EG1218-dk_Slide-Switches
- D0, D1, D2, D3, Q0, Q1, Q2, Q3: footprint LED_THT:LED_D3.0mm_Horizontal_O3.81mm_Z2.0mm -> custom:Emitter
Connections:
- net labels added: VCC, V_MOTOR
- net labels removed: M2_END_A, V_SRC
- wire segments 290 -> 296
- no-connect marks 9 -> 13
Other:
- note added: "* Resistors here act as current limiting resistors. Check that the resistor\n value properly limits current. Check the bluepills current limit for gpio"
- note removed: "Emitter / Receiver"
- moved on the sheet: BT1, BT_MH1, BT_MH2, C1, C10, C2, C9, R22, R23, S1, SK1, SK2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

Commit message: a
Parts:
- added C11: 10uF, Capacitor_SMD:C_1206_3216Metric_Pad1.33x1.80mm_HandSolder, symbol Device:C
- added C12, C13, C19: 0.1uF, Capacitor_SMD:C_1206_3216Metric_Pad1.33x1.80mm_HandSolder, symbol Device:C
- added C16: 100uF, Capacitor_THT:CP_Radial_D6.3mm_P2.50mm, symbol Device:C
- added C17, C18: 1uF, Capacitor_SMD:C_1206_3216Metric_Pad1.33x1.80mm_HandSolder, symbol Device:C
- added JP4, JP5: Jumper_2_Open, symbol Jumper:Jumper_2_Open
- added M3: M1_Conn_Alt, Connector_PinHeader_2.54mm:PinHeader_1x06_P2.54mm_Vertical, symbol Connector:Conn_01x06_Female
- added M4: M2_Conn_Alt, Connector_PinHeader_2.54mm:PinHeader_1x06_P2.54mm_Vertical, symbol Connector:Conn_01x06_Female
- added R12: 47K, Resistor_SMD:R_1206_3216Metric_Pad1.30x1.75mm_HandSolder, symbol Device:R
- added SW_RST1: SW, Button_Switch_THT:SW_PUSH_6mm, symbol Switch:SW_Push
- added TP3: TP_5V, Connector_PinHeader_2.54mm:PinHeader_1x01_P2.54mm_Vertical, symbol Connector:TestPoint
- added TP4: TP_3V3, Connector_PinHeader_2.54mm:PinHeader_1x01_P2.54mm_Vertical, symbol Connector:TestPoint
- added U4: APE8865Y5-33-HF-3, Package_TO_SOT_SMD:SOT-23-5, symbol Regulator_Linear:APE8865Y5-33-HF-3
- C1: value 100uF -> 0.1uF
- C10, C9: footprint Capacitor_SMD:C_1206_3216Metric_Pad1.42x1.75mm_HandSolder -> Capacitor_SMD:C_1206_3216Metric_Pad1.33x1.80mm_HandSolder
- M1, M2: footprint Connector_PinHeader_1.00mm:PinHeader_1x06_P1.00mm_Vertical -> Connector_JST:JST_SH_BM06B-SRSS-TB_1x06-1MP_P1.00mm_Vertical
- R11: value 10K -> 47K
Connections:
- net +3V3: now also R19.2, R20.2, R21.2, C11.1, C12.1, C18.1, M3.3 (Pin_3), M4.3 (Pin_3), R12.1, TP4.1, U4.5 (VOUT); no longer J4.1 (VTref), J5.1 (Pin_1), U1.20 (3V3), U1.38 (3V3)
- net +5V: now also C13.1, C16.1, C17.1, TP3.1, U4.1 (VIN), U4.3 (~SHDN~)
- net GND: now also C11.2, C12.2, C13.2, C16.2, C17.2, C18.2, C19.2, JP4.1 (A), JP5.2 (B), M3.6 (Pin_6), M4.6 (Pin_6), SW_RST1.2, U4.2 (GND); no longer D4.1 (K), D5.1 (K), D6.1 (K), R1.1, R2.1, R3.1, R4.1, U2.12 (GND), U2.13 (GND), U2.4 (GND), U2.5 (GND)
- net LED_BLUE: now also D6.1 (K); no longer R21.2
- net LED_GREEN: now also D5.1 (K); no longer R20.2
- net LED_RED: now also D4.1 (K); no longer R19.2
- net M1_ENC_A: now also M4.4 (Pin_4)
- net M1_ENC_B: now also M4.5 (Pin_5)
- net M1_OUT_1: now also M4.1 (Pin_1)
- net M1_OUT_2: now also M4.2 (Pin_2)
- net M2_ENC_A: now also M3.4 (Pin_4)
- net M2_ENC_B: now also M3.5 (Pin_5)
- net M2_OUT_1: now also M3.1 (Pin_1)
- net M2_OUT_2: now also M3.2 (Pin_2)
- net RST: now also C19.1, R12.2, SW_RST1.1
- new net 3V3_MCU: J4.1 (VTref), J5.1 (Pin_1), U1.20 (3V3), U1.38 (3V3)
- new net AGND: JP4.2 (B), R1.1, R2.1, R3.1, R4.1
- new net MGND: JP5.1 (A), U2.12 (GND), U2.13 (GND), U2.4 (GND), U2.5 (GND)
- no-connect marks 13 -> 14
Other:
- moved on the sheet: C2, C3, C4, C9, D4, D5, D6, M1, M2, MH1, MH2, R11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

Commit message: started work on pcb
Parts:
- added L1: 10uH, Inductor_SMD:L_1206_3216Metric_Pad1.42x1.75mm_HandSolder, symbol Device:L
- C1: footprint Capacitor_THT:CP_Radial_D6.3mm_P2.50mm -> Capacitor_SMD:C_1206_3216Metric_Pad1.33x1.80mm_HandSolder
- JP4, JP5: footprint (none) -> Jumper:SolderJumper-2_P1.3mm_Bridged_Pad1.0x1.5mm
- SW1, SW_RST1: footprint Button_Switch_THT:SW_PUSH_6mm -> Button_Switch_SMD:SW_SPST_REED_CT05-XXXX-G1
Connections:
- net +3V3: now also M1.4 (Pin_4), M2.4 (Pin_4), U1.20 (3V3), U1.38 (3V3), L1.1; no longer M1.3 (Pin_3), M2.3 (Pin_3), Q0.1 (C), Q1.1 (C), Q2.1 (C), Q3.1 (C)
- net +5V: no longer U1.18 (5V)
- net 3V3_MCU: no longer U1.20 (3V3), U1.38 (3V3)
- net GND: now also M1.1 (Pin_1), M2.1 (Pin_1); no longer M1.6 (Pin_6), M2.6 (Pin_6)
- net M1_ENC_A: now also M2.3 (Pin_3); no longer M2.4 (Pin_4)
- net M1_ENC_B: now also M2.2 (Pin_2); no longer M2.5 (Pin_5)
- net M1_OUT_1: now also M2.6 (Pin_6); no longer M2.1 (Pin_1)
- net M1_OUT_2: now also M2.5 (Pin_5); no longer M2.2 (Pin_2)
- net M2_ENC_A: now also M1.3 (Pin_3); no longer M1.4 (Pin_4)
- net M2_ENC_B: now also M1.2 (Pin_2); no longer M1.5 (Pin_5)
- net M2_OUT_1: now also M1.6 (Pin_6); no longer M1.1 (Pin_1)
- net M2_OUT_2: now also M1.5 (Pin_5); no longer M1.2 (Pin_2)
- new net +3.3VA: L1.2, Q0.1 (C), Q1.1 (C), Q2.1 (C), Q3.1 (C)
- no-connect marks 14 -> 15
Changed lines of the file:
@@
 	1    0    0    -1
 $EndComp
-$Comp
-L power:+5V #PWR0103
-U 1 1 63294D3E
-P 8525 1475
-F 0 "#PWR0103" H 8525 1325 50  0001 C CNN
-F 1 "+5V" H 8540 1648 50  0000 C CNN
-F 2 "" H 8525 1475 50  0001 C CNN
-F 3 "" H 8525 1475 50  0001 C CNN
-	1    8525 1475
-	1    0    0    -1
-$EndComp
-Wire Wire Line
-	8525 1475 8525 1675
 Text GLabel 9725 2075 2    50   Input ~ 0
 EMIT_4
@@
 RECEIV_4
 $Comp
-L power:+3V3 #PWR0108
-U 1 1 635C6453
-P 5135 2980
-F 0 "#PWR0108" H 5135 2830 50  0001 C CNN
-F 1 "+3V3" H 5150 3153 50  0000 C CNN
-F 2 "" H 5135 2980 50  0001 C CNN
-F 3 "" H 5135 2980 50  0001 C CNN
-	1    5135 2980
-	1    0    0    -1
-$EndComp
-$Comp
 L Device:C C1
 U 1 1 63609FB9
@@
 F 0 "C1" H 3290 7021 50  0000 L CNN
 F 1 "0.1uF" H 3290 6930 50  0000 L CNN
-F 2 "Capacitor_THT:CP_Radial_D6.3mm_P2.50mm" H 3213 6825 50  0001 C CNN
+F 2 "Capacitor_SMD:C_1206_3216Metric_Pad1.33x1.80mm_HandSolder" H 3213 6825 50  0001 C CNN
 F 3 "~" H 3175 6975 50  0001 C CNN
 	1    3175 6975
@@
 	1    0    0    -1
 $EndComp
-Text GLabel 14400 4225 0    50   Input ~ 0
+Text GLabel 14400 4125 0    50   Input ~ 0
 M1_ENC_A
+Text GLabel 14400 4025 0    50   Input ~ 0
+M1_ENC_B
+Text GLabel 14400 4425 0    50   Input ~ 0
+M1_OUT_1
 Text GLabel 14400 4325 0    50   Input ~ 0
-M1_ENC_B
-Text GLabel 14400 3925 0    50   Input ~ 0
-M1_OUT_1
-Text GLabel 14400 4025 0    50   Input ~ 0
 M1_OUT_2
-Wire Wire Line
-	13850 4425 13850 4625
-Wire Wire Line
-	13850 4425 14400 4425
 $Comp
 L power:GND #PWR0123
 U 1 1 63D93050
-P 13850 4625
-F 0 "#PWR0123" H 13850 4375 50  0001 C CNN
-F 1 "GND" H 13855 4452 50  0000 C CNN
-F 2 "" H 13850 4625 50  0001 C CNN
-F 3 "" H 13850 4625 50  0001 C CNN
-	1    13850 4625
-	1    0    0    -1
+P 14200 3800
+F 0 "#PWR0123" H 14200 3550 50  0001 C CNN
+F 1 "GND" H 14205 3627 50  0000 C CNN
+F 2 "" H 14200 3800 50  0001 C CNN
+F 3 "" H 14200 3800 50  0001 C CNN
+	1    14200 3800
+	-1   0    0    1
 $EndComp
 $Comp
@@
 	1    0    0    -1
 $EndComp
-Text GLabel 11800 4300 0    50   Input ~ 0
+Text GLabel 11800 4200 0    50   Input ~ 0
 M2_ENC_A
+Text GLabel 11800 4100 0    50   Input ~ 0
+M2_ENC_B
+Text GLabel 11800 4500 0    50   Input ~ 0
+M2_OUT_1
 Text GLabel 11800 4400 0    50   Input ~ 0
-M2_ENC_B
-Text GLabel 11800 4000 0    50   Input ~ 0
-M2_OUT_1
-Text GLabel 11800 4100 0    50   Input ~ 0
 M2_OUT_2
-Wire Wire Line
-	11250 4500 11250 4700
-Wire Wire Line
-	11250 4500 11800 4500
 $Comp
 L power:GND #PWR0125
 U 1 1 63DAFBE7
-P 11250 4700
-F 0 "#PWR0125" H 11250 4450 50  0001 C CNN
-F 1 "GND" H 11255 4527 50  0000 C CNN
-F 2 "" H 11250 4700 50  0001 C CNN
-F 3 "" H 11250 4700 50  0001 C CNN
-	1    11250 4700
-	1    0    0    -1
+P 11550 3850
+F 0 "#PWR0125" H 11550 3600 50  0001 C CNN
+F 1 "GND" H 11555 3677 50  0000 C CNN
+F 2 "" H 11550 3850 50  0001 C CNN
+F 3 "" H 11550 3850 50  0001 C CNN
+	1    11550 3850
+	-1   0    0    1
 $EndComp
 Wire Notes Line
@@
 F 0 "SW1" H 3775 9560 50  0000 C CNN
 F 1 "SW" H 3775 9469 50  0000 C CNN
-F 2 "Button_Switch_THT:SW_PUSH_6mm" H 3775 9475 50  0001 C CNN
+F 2 "Button_Switch_SMD:SW_SPST_REED_CT05-XXXX-G1" H 3775 9475 50  0001 C CNN
 F 3 "~" H 3775 9475 50  0001 C CNN
 	1    3775 9275
@@
 	-1   0    0    1
 $EndComp
-Wire Wire Line
-	14400 4125 13875 4125
-Wire Wire Line
-	13875 4125 13875 3800
-Wire Wire Line
-	11800 4200 11275 4200
-Wire Wire Line
-	11275 4200 11275 3900
 $Comp
 L power:+3V3 #PWR0124
@@
 Wire Wire Line
 	8725 1550 8725 1675
-Wire Wire Line
-	8725 1550 8950 1550
 Connection ~ 8725 1550
-Text GLabel 8950 1550 2    50   Input ~ 0
-3V3_MCU
 Text GLabel 8975 5575 2    50   Input ~ 0
 3V3_MCU
@@
 F 0 "SW_RST1" H 3750 10935 50  0000 C CNN
 F 1 "SW" H 3750 10844 50  0000 C CNN
-F 2 "Button_Switch_THT:SW_PUSH_6mm" H 3750 10850 50  0001 C CNN
+F 2 "Button_Switch_SMD:SW_SPST_REED_CT05-XXXX-G1" H 3750 10850 50  0001 C CNN
 F 3 "~" H 3750 10850 50  0001 C CNN
 	1    3750 10650
@@
 F 0 "JP5" H 14700 3535 50  0000 C CNN
 F 1 "Jumper_2_Open" H 14700 3444 50  0000 C CNN
-F 2 "" H 14700 3300 50  0001 C CNN
+F 2 "Jumper:SolderJumper-2_P1.3mm_Bridged_Pad1.0x1.5mm" H 14700 3300 50  0001 C CNN
 F 3 "~" H 14700 3300 50  0001 C CNN
 	1    14700 3300
@@
 F 0 "JP4" H 5775 7810 50  0000 C CNN
 F 1 "Jumper_2_Open" H 5775 7719 50  0000 C CNN
-F 2 "" H 5775 7575 50  0001 C CNN
+F 2 "Jumper:SolderJumper-2_P1.3mm_Bridged_Pad1.0x1.5mm" H 5775 7575 50  0001 C CNN
 F 3 "~" H 5775 7575 50  0001 C CNN
 	1    5775 7575
@@
 Text GLabel 5100 4400 3    50   Input ~ 0
 AGND
+Wire Wire Line
+	11800 4300 11275 4300
+Wire Wire Line
+	11275 4300 11275 3900
+Wire Wire Line
+	11800 4000 11550 4000
+Wire Wire Line
+	11550 4000 11550 3850
+Wire Wire Line
+	14400 4225 13875 4225
+Wire Wire Line
+	13875 4225 13875 3800
+Wire Wire Line
+	14400 3925 14200 3925
+Wire Wire Line
+	14200 3925 14200 3800
+$Comp
+L Device:L L1
+U 1 1 63514CF0
+P 5600 5375
+F 0 "L1" V 5790 5375 50  0000 C CNN
+F 1 "10uH" V 5699 5375 50  0000 C CNN
+F 2 "Inductor_SMD:L_1206_3216Metric_Pad1.42x1.75mm_HandSolder" H 5600 5375 50  0001 C CNN
+F 3 "~" H 5600 5375 50  0001 C CNN
+	1    5600 5375
+	0    -1   -1   0
+$EndComp
+$Comp
+L power:+3.3VA #PWR0103
+U 1 1 63517883
+P 6325 5225
+F 0 "#PWR0103" H 6325 5075 50  0001 C CNN
+F 1 "+3.3VA" H 6340 5398 50  0000 C CNN
+F 2 "" H 6325 5225 50  0001 C CNN
+F 3 "" H 6325 5225 50  0001 C CNN
+	1    6325 5225
+	1    0    0    -1
+$EndComp
+Wire Wire Line
+	6325 5225 6325 5375
+Wire Wire Line
+	6325 5375 5750 5375
+Wire Wire Line
+	5450 5375 4775 5375
+Connection ~ 4775 5375
+$Comp
+L power:+3.3VA #PWR0108
+U 1 1 6357E45C
+P 5135 2980
+F 0 "#PWR0108" H 5135 2830 50  0001 C CNN
+F 1 "+3.3VA" H 5150 3153 50  0000 C CNN
+F 2 "" H 5135 2980 50  0001 C CNN
+F 3 "" H 5135 2980 50  0001 C CNN
+	1    5135 2980
+	1    0    0    -1
+$EndComp
+NoConn ~ 8525 1675
+Wire Wire Line
+	9000 1550 9000 1350
+Wire Wire Line
+	8725 1550 9000 1550
+$Comp
+L power:+3V3 #PWR0122
+U 1 1 636F67AC
+P 9000 1350
+F 0 "#PWR0122" H 9000 1200 50  0001 C CNN
+F 1 "+3V3" H 9015 1523 50  0000 C CNN
+F 2 "" H 9000 1350 50  0001 C CNN
+F 3 "" H 9000 1350 50  0001 C CNN
+	1    9000 1350
+	1    0    0    -1
+$EndComp
 $EndSCHEMATC

Commit message: more tracing
Connections:
- net 3V3_MCU is gone; now on net +3V3: J4.1 (VTref), J5.1 (Pin_1)
- net BUTTON: now also U1.8 (PA11); no longer U1.5 (PA8)
- net EMIT_1: now also U1.1 (PB12); no longer U1.9 (PA12)
- net EMIT_2: now also U1.36 (PB11); no longer U1.8 (PA11)
- net EMIT_3: now also U1.13 (PB5); no longer U1.10 (PA15)
- net EMIT_4: now also U1.35 (PB10); no longer U1.36 (PB11)
- net LED_BLUE: now also U1.9 (PA12); no longer U1.35 (PB10)
- net LED_RED: now also U1.10 (PA15); no longer U1.13 (PB5)
- net M1_BACK: now also U1.3 (PB14); no longer U1.2 (PB13)
- net M1_ENC_A: now also U1.32 (PA7); no longer U1.15 (PB7)
- net M1_ENC_B: now also U1.31 (PA6); no longer U1.14 (PB6)
- net M1_FWD: now also U1.5 (PA8); no longer U1.1 (PB12)
- net M1_SPD: now also U1.17 (PB9); no longer U1.16 (PB8)
- net M2_ENC_A: now also U1.15 (PB7); no longer U1.31 (PA6)
- net M2_ENC_B: now also U1.14 (PB6); no longer U1.32 (PA7)
- net M2_FWD: now also U1.2 (PB13); no longer U1.3 (PB14)
- net M2_SPD: now also U1.16 (PB8); no longer U1.17 (PB9)
- net RECEIV_1: now also U1.30 (PA5); no longer U1.29 (PA4)
- net RECEIV_2: now also U1.29 (PA4); no longer U1.30 (PA5)
Changed lines of the file:
@@
 	1    0    0    -1
 $EndComp
-Text GLabel 7625 2775 0    50   Input ~ 0
+Text GLabel 7575 1975 0    50   Input ~ 0
 EMIT_1
-Text GLabel 7625 2675 0    50   Input ~ 0
+Text GLabel 9725 2075 2    50   Input ~ 0
 EMIT_2
 Text GLabel 7775 2575 0    50   Input ~ 0
@@
 Text GLabel 7775 2475 0    50   Input ~ 0
 USART1_TX
-Text GLabel 7650 2375 0    50   Input ~ 0
+Text GLabel 7650 2675 0    50   Input ~ 0
 BUTTON
-Text GLabel 7700 2275 0    50   Input ~ 0
+Text GLabel 7675 2275 0    50   Input ~ 0
 M2_BACK
-Text GLabel 7650 2175 0    50   Input ~ 0
+Text GLabel 7625 2075 0    50   Input ~ 0
 M2_FWD
-Text GLabel 7700 2075 0    50   Input ~ 0
+Text GLabel 7675 2175 0    50   Input ~ 0
 M1_BACK
-Text GLabel 7650 1975 0    50   Input ~ 0
+Text GLabel 7625 2375 0    50   Input ~ 0
 M1_FWD
 Wire Wire Line
@@
 	1    0    0    -1
 $EndComp
-Text GLabel 9725 2075 2    50   Input ~ 0
+Text GLabel 9750 2175 2    50   Input ~ 0
 EMIT_4
-Text GLabel 9625 2175 2    50   Input ~ 0
+Text GLabel 7725 2775 0    50   Input ~ 0
 LED_BLUE
 Text GLabel 9650 2275 2    50   Input ~ 0
@@
 Text GLabel 9650 2375 2    50   Input ~ 0
 RECEIV_3
-Text GLabel 9600 2475 2    50   Input ~ 0
+Text GLabel 7725 3275 0    50   Input ~ 0
 M2_ENC_B
-Text GLabel 9600 2575 2    50   Input ~ 0
+Text GLabel 7725 3375 0    50   Input ~ 0
 M2_ENC_A
+Text GLabel 9625 2775 2    50   Input ~ 0
+RECEIV_2
 Text GLabel 9625 2675 2    50   Input ~ 0
-RECEIV_2
-Text GLabel 9625 2775 2    50   Input ~ 0
 RECEIV_1
 Text GLabel 9575 2875 2    50   Input ~ 0
@@
 Text GLabel 9675 3175 2    50   Input ~ 0
 BUZZER
-Text GLabel 7625 2875 0    50   Input ~ 0
+Text GLabel 7600 3175 0    50   Input ~ 0
 EMIT_3
 Text GLabel 7775 3075 0    50   Input ~ 0
 LED_GREEN
-Text GLabel 7675 3175 0    50   Input ~ 0
+Text GLabel 7700 2875 0    50   Input ~ 0
 LED_RED
-Text GLabel 7725 3275 0    50   Input ~ 0
+Text GLabel 9600 2575 2    50   Input ~ 0
 M1_ENC_B
-Text GLabel 7725 3375 0    50   Input ~ 0
+Text GLabel 9600 2475 2    50   Input ~ 0
 M1_ENC_A
+Text GLabel 7650 3575 0    50   Input ~ 0
+M1_SPD
 Text GLabel 7650 3475 0    50   Input ~ 0
-M1_SPD
-Text GLabel 7650 3575 0    50   Input ~ 0
 M2_SPD
 Text GLabel 9850 1975 2    50   Input ~ 0
@@
 SWO
 Wire Wire Line
-	7825 1975 7650 1975
-Wire Wire Line
-	7825 2075 7700 2075
-Wire Wire Line
-	7825 2175 7650 2175
-Wire Wire Line
-	7825 2275 7700 2275
-Wire Wire Line
-	7825 2375 7650 2375
-Wire Wire Line
 	7825 2475 7775 2475
 Wire Wire Line
 	7825 2575 7775 2575
 Wire Wire Line
-	7825 2675 7625 2675
-Wire Wire Line
-	7825 2775 7625 2775
-Wire Wire Line
-	7825 2875 7625 2875
-Wire Wire Line
 	7825 3075 7775 3075
-Wire Wire Line
-	7825 3175 7675 3175
 Wire Wire Line
 	7825 3275 7725 3275
@@
 Wire Wire Line
 	9425 2075 9725 2075
-Wire Wire Line
-	9425 2175 9625 2175
 Wire Wire Line
 	9425 2475 9600 2475
@@
 	8725 1550 8725 1675
 Connection ~ 8725 1550
-Text GLabel 8975 5575 2    50   Input ~ 0
-3V3_MCU
 Wire Wire Line
 	8525 5575 8975 5575
-Text GLabel 8200 6525 2    50   Input ~ 0
-3V3_MCU
 $Comp
 L Regulator_Linear:APE8865Y5-33-HF-3 U4
@@
 	1    0    0    -1
 $EndComp
+$Comp
+L power:+3V3 #PWR0149
+U 1 1 635D6435
+P 8975 5500
+F 0 "#PWR0149" H 8975 5350 50  0001 C CNN
+F 1 "+3V3" H 8990 5673 50  0000 C CNN
+F 2 "" H 8975 5500 50  0001 C CNN
+F 3 "" H 8975 5500 50  0001 C CNN
+	1    8975 5500
+	1    0    0    -1
+$EndComp
+$Comp
+L power:+3V3 #PWR0150
+U 1 1 635D6DA4
+P 8200 6525
+F 0 "#PWR0150" H 8200 6375 50  0001 C CNN
+F 1 "+3V3" H 8215 6698 50  0000 C CNN
+F 2 "" H 8200 6525 50  0001 C CNN
+F 3 "" H 8200 6525 50  0001 C CNN
+	1    8200 6525
+	1    0    0    -1
+$EndComp
+Wire Wire Line
+	8975 5575 8975 5500
+Wire Wire Line
+	7825 2875 7700 2875
+Wire Wire Line
+	7600 3175 7825 3175
+Wire Wire Line
+	9425 2175 9750 2175
+Wire Wire Line
+	7825 2775 7725 2775
+Wire Wire Line
+	7825 2675 7650 2675
+Wire Wire Line
+	7575 1975 7825 1975
+Wire Wire Line
+	7825 2075 7625 2075
+Wire Wire Line
+	7675 2175 7825 2175
+Wire Wire Line
+	7825 2275 7675 2275
+Wire Wire Line
+	7625 2375 7825 2375
 $EndSCHEMATC
