File: mouse_v2.sch (KiCad schematic (older format))
At the start: 98 parts, among them J1 HC05 Header, J2 Serial Debug Header, J3 HC05_Key Jump, J4 Conn_ARM_JTAG_SWD_10, J5 SWD Header, M1 M1_Conn, M2 M2_Conn, M3 M1_Conn_Alt, M4 M2_Conn_Alt, Q0 Q_Photo_NPN, Q1 Q_Photo_NPN, Q2 Q_Photo_NPN, Q3 Q_Photo_NPN, Q4 Q_NMOS_SGD, Q5 Q_NMOS_SGD, Q6 Q_NMOS_SGD, Q7 Q_NMOS_SGD, Q8 Q_NMOS_SGD, SW1 SW, U1 YAAJ_BluePill_SWD_Breakout, U2 L293D, U3 LM1085-5.0, U4 APE8865Y5-33-HF-3

Commit message: tracing
Parts:
- added J6, J7, J8, J9: Conn_01x02_Female, Connector_PinSocket_2.00mm:PinSocket_1x02_P2.00mm_Vertical, symbol Connector:Conn_01x02_Female
Connections:
- net AGND: now also J6.2 (Pin_2), J7.2 (Pin_2), J8.2 (Pin_2), J9.2 (Pin_2)
- net BUTTON: now also U1.12 (PB4); no longer U1.8 (PA11)
- net LED_GREEN: now also U1.10 (PA15); no longer U1.12 (PB4)
- net LED_RED: now also U1.8 (PA11); no longer U1.10 (PA15)
- net M1_ENC_A: now also U1.31 (PA6); no longer U1.32 (PA7)
- net M1_ENC_B: now also U1.32 (PA7); no longer U1.31 (PA6)
- net RECEIV_1: now also J6.1 (Pin_1)
- net RECEIV_2: now also J7.1 (Pin_1)
- net RECEIV_3: now also J8.1 (Pin_1)
- net RECEIV_4: now also J9.1 (Pin_1)
Changed lines of the file:
@@
 Text GLabel 7775 2475 0    50   Input ~ 0
 USART1_TX
-Text GLabel 7650 2675 0    50   Input ~ 0
+Text GLabel 7625 3075 0    50   Input ~ 0
 BUTTON
 Text GLabel 7675 2275 0    50   Input ~ 0
@@
 Text GLabel 7600 3175 0    50   Input ~ 0
 EMIT_3
-Text GLabel 7775 3075 0    50   Input ~ 0
+Text GLabel 7750 2875 0    50   Input ~ 0
 LED_GREEN
-Text GLabel 7700 2875 0    50   Input ~ 0
+Text GLabel 7650 2675 0    50   Input ~ 0
 LED_RED
+Text GLabel 9600 2475 2    50   Input ~ 0
+M1_ENC_B
 Text GLabel 9600 2575 2    50   Input ~ 0
-M1_ENC_B
-Text GLabel 9600 2475 2    50   Input ~ 0
 M1_ENC_A
 Text GLabel 7650 3575 0    50   Input ~ 0
@@
 	7825 2575 7775 2575
 Wire Wire Line
-	7825 3075 7775 3075
-Wire Wire Line
 	7825 3275 7725 3275
 Wire Wire Line
@@
 Wire Wire Line
 	5020 4345 5100 4345
-Wire Wire Line
-	5100 4345 5100 4405
 Connection ~ 5020 4345
 $Comp
@@
 Wire Wire Line
 	6100 7575 5975 7575
-Text GLabel 5100 4400 3    50   Input ~ 0
+Text GLabel 5100 4425 3    50   Input ~ 0
 AGND
 Wire Wire Line
@@
 	8975 5575 8975 5500
 Wire Wire Line
-	7825 2875 7700 2875
-Wire Wire Line
 	7600 3175 7825 3175
 Wire Wire Line
@@
 	7825 2775 7725 2775
 Wire Wire Line
+	7575 1975 7825 1975
+Wire Wire Line
+	7825 2075 7625 2075
+Wire Wire Line
+	7675 2175 7825 2175
+Wire Wire Line
+	7825 2275 7675 2275
+Wire Wire Line
+	7625 2375 7825 2375
+$Comp
+L Connector:Conn_01x02_Female J6
+U 1 1 635B9403
+P 1075 3850
+F 0 "J6" H 1103 3826 50  0000 L CNN
+F 1 "Conn_01x02_Female" H 1103 3735 50  0000 L CNN
+F 2 "Connector_PinSocket_2.00mm:PinSocket_1x02_P2.00mm_Vertical" H 1075 3850 50  0001 C CNN
+F 3 "~" H 1075 3850 50  0001 C CNN
+	1    1075 3850
+	1    0    0    -1
+$EndComp
+$Comp
+L Connector:Conn_01x02_Female J7
+U 1 1 635BB2ED
+P 1075 4050
+F 0 "J7" H 1103 4026 50  0000 L CNN
+F 1 "Conn_01x02_Female" H 1103 3935 50  0000 L CNN
+F 2 "Connector_PinSocket_2.00mm:PinSocket_1x02_P2.00mm_Vertical" H 1075 4050 50  0001 C CNN
+F 3 "~" H 1075 4050 50  0001 C CNN
+	1    1075 4050
+	1    0    0    -1
+$EndComp
+$Comp
+L Connector:Conn_01x02_Female J8
+U 1 1 635BB64C
+P 1075 4275
+F 0 "J8" H 1103 4251 50  0000 L CNN
+F 1 "Conn_01x02_Female" H 1103 4160 50  0000 L CNN
+F 2 "Connector_PinSocket_2.00mm:PinSocket_1x02_P2.00mm_Vertical" H 1075 4275 50  0001 C CNN
+F 3 "~" H 1075 4275 50  0001 C CNN
+	1    1075 4275
+	1    0    0    -1
+$EndComp
+$Comp
+L Connector:Conn_01x02_Female J9
+U 1 1 635BBA41
+P 1075 4500
+F 0 "J9" H 1103 4476 50  0000 L CNN
+F 1 "Conn_01x02_Female" H 1103 4385 50  0000 L CNN
+F 2 "Connector_PinSocket_2.00mm:PinSocket_1x02_P2.00mm_Vertical" H 1075 4500 50  0001 C CNN
+F 3 "~" H 1075 4500 50  0001 C CNN
+	1    1075 4500
+	1    0    0    -1
+$EndComp
+Text GLabel 875  3850 0    50   Input ~ 0
+RECEIV_1
+Text GLabel 875  4050 0    50   Input ~ 0
+RECEIV_2
+Text GLabel 875  4275 0    50   Input ~ 0
+RECEIV_3
+Text GLabel 875  4500 0    50   Input ~ 0
+RECEIV_4
+Text GLabel 875  3950 0    50   Input ~ 0
+AGND
+Text GLabel 875  4150 0    50   Input ~ 0
+AGND
+Text GLabel 875  4375 0    50   Input ~ 0
+AGND
+Text GLabel 875  4600 0    50   Input ~ 0
+AGND
+Wire Wire Line
+	5100 4345 5100 4425
+Wire Wire Line
+	7625 3075 7825 3075
+Wire Wire Line
+	7750 2875 7825 2875
+Wire Wire Line
 	7825 2675 7650 2675
-Wire Wire Line
-	7575 1975 7825 1975
-Wire Wire Line
-	7825 2075 7625 2075
-Wire Wire Line
-	7675 2175 7825 2175
-Wire Wire Line
-	7825 2275 7675 2275
-Wire Wire Line
-	7625 2375 7825 2375
 $EndSCHEMATC

Commit message: tracing
Parts:
- removed JP5: Jumper_2_Open, Jumper:SolderJumper-2_P1.3mm_Bridged_Pad1.0x1.5mm, symbol Jumper:Jumper_2_Open
- added C14, C15, C20, C21: 1uF, Capacitor_SMD:C_1206_3216Metric_Pad1.33x1.80mm_HandSolder, symbol Device:C
Connections:
- net MGND is gone; now on net GND: U2.12 (GND), U2.13 (GND), U2.4 (GND), U2.5 (GND)
- net +3.3VA: now also C14.1, C15.1, C20.1, C21.1
- net AGND: now also C14.2, C15.2, C20.2, C21.2
- net GND: now also C2.2; no longer C2.1
- net VCC: now also C2.1; no longer C2.2
Changed lines of the file:
@@
 Comment4 ""
 $EndDescr
-Wire Wire Line
-	5020 3045 4120 3045
 $Comp
 L mouse_v2-rescue:Q_Photo_NPN-Device Q0
@@
 Text GLabel 7775 2475 0    50   Input ~ 0
 USART1_TX
-Text GLabel 7625 3075 0    50   Input ~ 0
-BUTTON
 Text GLabel 7675 2275 0    50   Input ~ 0
 M2_BACK
@@
 M1_FWD
 Wire Wire Line
-	8625 3875 8625 3975
-Wire Wire Line
 	8625 3975 8525 3975
 Wire Wire Line
-	8525 3975 8525 3875
-Wire Wire Line
 	8525 3975 8425 3975
-Wire Wire Line
-	8425 3975 8425 3875
 Connection ~ 8525 3975
 Wire Wire Line
@@
 Text GLabel 7600 3175 0    50   Input ~ 0
 EMIT_3
-Text GLabel 7750 2875 0    50   Input ~ 0
-LED_GREEN
-Text GLabel 7650 2675 0    50   Input ~ 0
-LED_RED
-Text GLabel 9600 2475 2    50   Input ~ 0
-M1_ENC_B
-Text GLabel 9600 2575 2    50   Input ~ 0
-M1_ENC_A
 Text GLabel 7650 3575 0    50   Input ~ 0
 M1_SPD
@@
 	3220 3595 3220 3710
 Wire Wire Line
-	5020 3045 5135 3045
-Wire Wire Line
 	5135 3045 5135 2980
-Connection ~ 5020 3045
 Wire Wire Line
 	2370 3595 2370 3735
@@
 Wire Wire Line
 	3650 7200 3175 7200
-$Comp
-L Device:C C2
-U 1 1 6362DC24
-P 2700 6975
-F 0 "C2" H 2815 7021 50  0000 L CNN
-F 1 "100uF" H 2815 6930 50  0000 L CNN
-F 2 "Capacitor_THT:CP_Radial_D6.3mm_P2.50mm" H 2738 6825 50  0001 C CNN
-F 3 "~" H 2700 6975 50  0001 C CNN
-	1    2700 6975
-	-1   0    0    1
-$EndComp
 Wire Wire Line
 	3175 7200 3175 7125
@@
 Wire Wire Line
 	4575 5375 4775 5375
-Text GLabel 13300 3375 3    50   Input ~ 0
-MGND
 Wire Wire Line
 	13300 3100 13300 3375
-Text GLabel 14300 3300 0    50   Input ~ 0
-MGND
-$Comp
-L power:GND #PWR0107
-U 1 1 6387BAF7
-P 15000 3425
-F 0 "#PWR0107" H 15000 3175 50  0001 C CNN
-F 1 "GND" H 15005 3252 50  0000 C CNN
-F 2 "" H 15000 3425 50  0001 C CNN
-F 3 "" H 15000 3425 50  0001 C CNN
-	1    15000 3425
-	1    0    0    -1
-$EndComp
-$Comp
-L Jumper:Jumper_2_Open JP5
-U 1 1 6387D303
-P 14700 3300
-F 0 "JP5" H 14700 3535 50  0000 C CNN
-F 1 "Jumper_2_Open" H 14700 3444 50  0000 C CNN
-F 2 "Jumper:SolderJumper-2_P1.3mm_Bridged_Pad1.0x1.5mm" H 14700 3300 50  0001 C CNN
-F 3 "~" H 14700 3300 50  0001 C CNN
-	1    14700 3300
-	1    0    0    -1
-$EndComp
-Wire Wire Line
-	15000 3425 15000 3300
-Wire Wire Line
-	15000 3300 14900 3300
-Wire Wire Line
-	14500 3300 14300 3300
 Wire Wire Line
 	5300 7200 5300 7575
@@
 AGND
 Wire Wire Line
-	5100 4345 5100 4425
+	5100 4345 5100 4350
+Wire Wire Line
+	7825 2675 7650 2675
+Text GLabel 9600 2475 2    50   Input ~ 0
+M1_ENC_B
+Text GLabel 9600 2575 2    50   Input ~ 0
+M1_ENC_A
+Text GLabel 7625 3075 0    50   Input ~ 0
+BUTTON
 Wire Wire Line
 	7625 3075 7825 3075
+Text GLabel 7650 2675 0    50   Input ~ 0
+LED_RED
+Text GLabel 7750 2875 0    50   Input ~ 0
+LED_GREEN
 Wire Wire Line
 	7750 2875 7825 2875
-Wire Wire Line
-	7825 2675 7650 2675
+$Comp
+L Device:C C2
+U 1 1 6362DC24
+P 2700 6975
+F 0 "C2" H 2450 6975 50  0000 L CNN
+F 1 "100uF" H 2400 6875 50  0000 L CNN
+F 2 "Capacitor_THT:CP_Radial_D6.3mm_P2.50mm" H 2738 6825 50  0001 C CNN
+F 3 "~" H 2700 6975 50  0001 C CNN
+	1    2700 6975
+	1    0    0    -1
+$EndComp
+$Comp
+L Device:C C14
+U 1 1 63609F53
+P 5450 3700
+F 0 "C14" H 5565 3746 50  0000 L CNN
+F 1 "1uF" H 5565 3655 50  0000 L CNN
+F 2 "Capacitor_SMD:C_1206_3216Metric_Pad1.33x1.80mm_HandSolder" H 5488 3550 50  0001 C CNN
+F 3 "~" H 5450 3700 50  0001 C CNN
+	1    5450 3700
+	1    0    0    -1
+$EndComp
+$Comp
+L Device:C C15
+U 1 1 6360A313
+P 5775 3700
+F 0 "C15" H 5890 3746 50  0000 L CNN
+F 1 "1uF" H 5890 3655 50  0000 L CNN
+F 2 "Capacitor_SMD:C_1206_3216Metric_Pad1.33x1.80mm_HandSolder" H 5813 3550 50  0001 C CNN
+F 3 "~" H 5775 3700 50  0001 C CNN
+	1    5775 3700
+	1    0    0    -1
+$EndComp
+$Comp
+L Device:C C20
+U 1 1 6360AA87
+P 6100 3700
+F 0 "C20" H 6215 3746 50  0000 L CNN
+F 1 "1uF" H 6215 3655 50  0000 L CNN
+F 2 "Capacitor_SMD:C_1206_3216Metric_Pad1.33x1.80mm_HandSolder" H 6138 3550 50  0001 C CNN
+F 3 "~" H 6100 3700 50  0001 C CNN
+	1    6100 3700
+	1    0    0    -1
+$EndComp
+$Comp
+L Device:C C21
+U 1 1 6360AE4E
+P 6400 3700
+F 0 "C21" H 6515 3746 50  0000 L CNN
+F 1 "1uF" H 6515 3655 50  0000 L CNN
+F 2 "Capacitor_SMD:C_1206_3216Metric_Pad1.33x1.80mm_HandSolder" H 6438 3550 50  0001 C CNN
+F 3 "~" H 6400 3700 50  0001 C CNN
+	1    6400 3700
+	1    0    0    -1
+$EndComp
+Wire Wire Line
+	5450 3550 5775 3550
+Connection ~ 5775 3550
+Wire Wire Line
+	5775 3550 5925 3550
+Connection ~ 6100 3550
+Wire Wire Line
+	6100 3550 6400 3550
+Wire Wire Line
+	6400 3850 6100 3850
+Connection ~ 5775 3850
+Wire Wire Line
+	5775 3850 5450 3850
+Connection ~ 6100 3850
+Wire Wire Line
+	6100 3850 5925 3850
+Wire Wire Line
+	5925 3850 5925 4350
+Wire Wire Line
+	5925 4350 5100 4350
+Connection ~ 5925 3850
+Wire Wire Line
+	5925 3850 5775 3850
+Connection ~ 5100 4350
+Wire Wire Line
+	5100 4350 5100 4425
+Connection ~ 5925 3550
+Wire Wire Line
+	5925 3550 6100 3550
+Wire Wire Line
+	5925 3045 5925 3550
+Wire Wire Line
+	4120 3045 5020 3045
+Connection ~ 5020 3045
+Wire Wire Line
+	5020 3045 5135 3045
+Connection ~ 5135 3045
+Wire Wire Line
+	5135 3045 5925 3045
+$Comp
+L power:GND #PWR?
+U 1 1 63794FA2
+P 13300 3375
+F 0 "#PWR?" H 13300 3125 50  0001 C CNN
+F 1 "GND" H 13305 3202 50  0000 C CNN
+F 2 "" H 13300 3375 50  0001 C CNN
+F 3 "" H 13300 3375 50  0001 C CNN
+	1    13300 3375
+	1    0    0    -1
+$EndComp
 $EndSCHEMATC
