File: mouse_v2.sch (KiCad schematic (older format))
At the start: 105 parts, among them J1 HC05 Header, J2 Serial Debug Header, J3 HC05_Key Jump, J4 Conn_ARM_JTAG_SWD_10, J5 SWD Header, J6 Conn_01x02_Female, J7 Conn_01x02_Female, J8 Conn_01x02_Female, J9 Conn_01x02_Female, M1 M1_Conn, M2 M2_Conn, M3 M1_Conn_Alt, M4 M2_Conn_Alt, Q0 Q_Photo_NPN, Q1 Q_Photo_NPN, Q2 Q_Photo_NPN, Q3 Q_Photo_NPN, Q4 Q_NMOS_SGD, Q5 Q_NMOS_SGD, Q6 Q_NMOS_SGD, Q7 Q_NMOS_SGD, Q8 Q_NMOS_SGD, SW1 SW, U1 YAAJ_BluePill_SWD_Breakout, U2 L293D, U3 LM1085-5.0, U4 APE8865Y5-33-HF-3

Commit message: tracing
Parts:
- added Q10, Q11, Q12, Q9: Q_NMOS_GSD, Package_TO_SOT_SMD:SOT-23, symbol Device:Q_NMOS_GSD
- U3: footprint Package_TO_SOT_SMD:TO-263-3_TabPin2 -> custom:VREG_TO-263-3_TabPin2
Connections:
- net EMIT_1: now also Q9.1 (G)
- net EMIT_2: now also Q10.1 (G)
- net EMIT_3: now also Q11.1 (G)
- net EMIT_4: now also Q12.1 (G)
- net GND: now also Q10.2 (S), Q11.2 (S), Q12.2 (S), Q9.2 (S)
- net at Q7.3 (D), R8.2: now also Q12.3 (D)
- net at Q6.3 (D), R7.2: now also Q11.3 (D)
- net at Q4.3 (D), R5.2: now also Q9.3 (D)
- net at Q5.3 (D), R6.2: now also Q10.3 (D)
Changed lines of the file:
@@
 F 0 "U3" H 4225 6917 50  0000 C CNN
 F 1 "LM1085-5.0" H 4225 6826 50  0000 C CNN
-F 2 "Package_TO_SOT_SMD:TO-263-3_TabPin2" H 4225 6925 50  0001 C CIN
+F 2 "custom:VREG_TO-263-3_TabPin2" H 4225 6925 50  0001 C CIN
 F 3 "http://www.ti.com/lit/ds/symlink/lm1084.pdf" H 4225 6675 50  0001 C CNN
 	1    4225 6675
@@
 	900  2000 1000 2000
 Wire Wire Line
-	1300 1700 1300 1800
+	1300 1700 1300 1725
 Wire Wire Line
 	1300 1300 1300 1400
@@
 	3900 2000 4000 2000
 Wire Wire Line
-	4300 1700 4300 1800
+	4300 1700 4300 1750
 Wire Wire Line
 	4300 1300 4300 1400
@@
 Wire Wire Line
 	4000 2000 4000 2400
-Wire Wire Line
-	4300 2200 4300 2400
 $Comp
 L mouse_v2-rescue:IRL81A-LED D2
@@
 Wire Wire Line
 	5400 2000 5500 2000
-Wire Wire Line
-	5800 1700 5800 1800
 Wire Wire Line
 	5800 1300 5800 1400
@@
 	5135 3045 5925 3045
 $Comp
-L power:GND #PWR?
+L power:GND #PWR0107
 U 1 1 63794FA2
 P 13300 3375
-F 0 "#PWR?" H 13300 3125 50  0001 C CNN
+F 0 "#PWR0107" H 13300 3125 50  0001 C CNN
 F 1 "GND" H 13305 3202 50  0000 C CNN
 F 2 "" H 13300 3375 50  0001 C CNN
@@
 	1    0    0    -1
 $EndComp
+Wire Wire Line
+	6350 1925 6350 2200
+Wire Wire Line
+	6350 2200 5800 2200
+Connection ~ 5800 2200
+Wire Wire Line
+	5500 1725 5500 2000
+Wire Wire Line
+	4825 1525 4450 1525
+Wire Wire Line
+	4450 1525 4450 1750
+Wire Wire Line
+	4450 1750 4300 1750
+Connection ~ 4300 1750
+Wire Wire Line
+	4300 1750 4300 1800
+Wire Wire Line
+	4525 1725 4525 1875
+Wire Wire Line
+	4525 1875 4000 1875
+Wire Wire Line
+	4000 1875 4000 2000
+Wire Wire Line
+	4825 1925 4825 2325
+Wire Wire Line
+	4825 2325 4300 2325
+Wire Wire Line
+	4300 2200 4300 2325
+Connection ~ 4300 2325
+Wire Wire Line
+	4300 2325 4300 2400
+Wire Wire Line
+	3275 1950 3275 2200
+Wire Wire Line
+	3275 2200 2800 2200
+Connection ~ 2800 2200
+Wire Wire Line
+	2975 1750 2500 1750
+Wire Wire Line
+	2500 1750 2500 2000
+Wire Wire Line
+	3275 1550 3050 1550
+Wire Wire Line
+	3050 1550 3050 1700
+Wire Wire Line
+	3050 1700 2800 1700
+Connection ~ 2800 1700
+Wire Wire Line
+	1775 1575 1425 1575
+Wire Wire Line
+	1425 1575 1425 1725
+Wire Wire Line
+	1425 1725 1300 1725
+Connection ~ 1300 1725
+Wire Wire Line
+	1300 1725 1300 1800
+Wire Wire Line
+	1775 1975 1775 2400
+Wire Wire Line
+	1775 2400 1300 2400
+$Comp
+L Device:Q_NMOS_GSD Q12
+U 1 1 638F1AA4
+P 6250 1725
+F 0 "Q12" H 6454 1771 50  0000 L CNN
+F 1 "Q_NMOS_GSD" H 6454 1680 50  0000 L CNN
+F 2 "Package_TO_SOT_SMD:SOT-23" H 6450 1825 50  0001 C CNN
+F 3 "~" H 6250 1725 50  0001 C CNN
+	1    6250 1725
+	1    0    0    -1
+$EndComp
+$Comp
+L Device:Q_NMOS_GSD Q11
+U 1 1 638F34B2
+P 4725 1725
+F 0 "Q11" H 4929 1771 50  0000 L CNN
+F 1 "Q_NMOS_GSD" H 4929 1680 50  0000 L CNN
+F 2 "Package_TO_SOT_SMD:SOT-23" H 4925 1825 50  0001 C CNN
+F 3 "~" H 4725 1725 50  0001 C CNN
+	1    4725 1725
+	1    0    0    -1
+$EndComp
+$Comp
+L Device:Q_NMOS_GSD Q10
+U 1 1 638F43B8
+P 3175 1750
+F 0 "Q10" H 3379 1796 50  0000 L CNN
+F 1 "Q_NMOS_GSD" H 3379 1705 50  0000 L CNN
+F 2 "Package_TO_SOT_SMD:SOT-23" H 3375 1850 50  0001 C CNN
+F 3 "~" H 3175 1750 50  0001 C CNN
+	1    3175 1750
+	1    0    0    -1
+$EndComp
+$Comp
+L Device:Q_NMOS_GSD Q9
+U 1 1 638F50C4
+P 1675 1775
+F 0 "Q9" H 1879 1821 50  0000 L CNN
+F 1 "Q_NMOS_GSD" H 1879 1730 50  0000 L CNN
+F 2 "Package_TO_SOT_SMD:SOT-23" H 1875 1875 50  0001 C CNN
+F 3 "~" H 1675 1775 50  0001 C CNN
+	1    1675 1775
+	1    0    0    -1
+$EndComp
+Wire Wire Line
+	6050 1725 5500 1725
+Wire Wire Line
+	5800 1700 5800 1775
+Wire Wire Line
+	5800 1775 6000 1775
+Wire Wire Line
+	6000 1775 6000 1525
+Wire Wire Line
+	6000 1525 6350 1525
+Connection ~ 5800 1775
+Wire Wire Line
+	5800 1775 5800 1800
+Wire Wire Line
+	1000 1775 1000 2000
+Wire Wire Line
+	1000 1775 1475 1775
 $EndSCHEMATC

Commit message: v0 PCB
Parts:
- added C25: 10nF, Capacitor_SMD:C_1206_3216Metric_Pad1.33x1.80mm_HandSolder, symbol Device:C
Connections:
- net +3V3: now also U4.4 (BYP); no longer U4.5 (VOUT)
- net GND: now also C25.2
- new net 3V3_BYP: C25.1, U4.5 (VOUT)
- no-connect marks 15 -> 14
Other:
- note added: "On my reg VOUT and BYP swapped"
Changed lines of the file:
@@
 	1    0    0    -1
 $EndComp
-NoConn ~ 3275 5475
 Wire Wire Line
 	2225 5375 2225 5475
@@
 Wire Wire Line
 	2225 5375 1950 5375
-Wire Wire Line
-	3275 5375 3400 5375
 Wire Wire Line
 	3725 5375 3725 5200
@@
 	1    0    0    -1
 $EndComp
-Wire Wire Line
-	3400 5450 3400 5375
-Connection ~ 3400 5375
 Wire Wire Line
 	3400 5375 3725 5375
@@
 Wire Wire Line
 	1000 1775 1475 1775
+Wire Wire Line
+	3275 5475 3400 5475
+Wire Wire Line
+	3400 5375 3400 5450
+Connection ~ 3400 5450
+Wire Wire Line
+	3400 5450 3400 5475
+Text Notes 2975 5775 0    50   ~ 0
+On my reg VOUT and BYP swapped
+Wire Wire Line
+	3275 5375 3350 5375
+Wire Wire Line
+	3350 5375 3350 5275
+Wire Wire Line
+	3350 5275 3425 5275
+Text GLabel 3400 5050 0    50   Input ~ 0
+3V3_BYP
+Wire Wire Line
+	3425 5050 3400 5050
+Wire Wire Line
+	3425 5050 3425 5275
+Text GLabel 5675 5600 0    50   Input ~ 0
+3V3_BYP
+$Comp
+L Device:C C25
+U 1 1 63803AB5
+P 5800 5800
+F 0 "C25" H 5915 5846 50  0000 L CNN
+F 1 "10nF" H 5915 5755 50  0000 L CNN
+F 2 "Capacitor_SMD:C_1206_3216Metric_Pad1.33x1.80mm_HandSolder" H 5838 5650 50  0001 C CNN
+F 3 "~" H 5800 5800 50  0001 C CNN
+	1    5800 5800
+	1    0    0    -1
+$EndComp
+Wire Wire Line
+	5800 5650 5800 5600
+Wire Wire Line
+	5800 5600 5675 5600
+$Comp
+L power:GND #PWR0151
+U 1 1 63861CB5
+P 5800 6050
+F 0 "#PWR0151" H 5800 5800 50  0001 C CNN
+F 1 "GND" H 5805 5877 50  0000 C CNN
+F 2 "" H 5800 6050 50  0001 C CNN
+F 3 "" H 5800 6050 50  0001 C CNN
+	1    5800 6050
+	1    0    0    -1
+$EndComp
+Wire Wire Line
+	5800 5950 5800 6050
 $EndSCHEMATC

Commit message: changes for v0.1 wip
Parts:
- removed C5, C7: 22pF, Capacitor_SMD:C_0603_1608Metric_Pad1.08x0.95mm_HandSolder, symbol Device:C_Small
- removed FB1, FB2: HZ0603C601R-10, Resistor_SMD:R_0603_1608Metric_Pad0.98x0.95mm_HandSolder, symbol Device:FerriteBead_Small
- removed J2: Serial Debug Header, Connector_PinHeader_2.54mm:PinHeader_1x06_P2.54mm_Vertical, symbol Connector:Conn_01x06_Female
- removed J3: HC05_Key Jump, Connector_PinHeader_2.54mm:PinHeader_1x02_P2.54mm_Vertical, symbol Connector:Conn_01x02_Male
- J1: value HC05 Header -> Serial Debug Header
Connections:
- net HC05_Key is gone; now on net GND: J1.6 (Pin_6)
- net USART2_RX is gone; now on net M1_SPD: U1.28 (PA3)
- net USART2_TX is gone; now on net M2_SPD: U1.27 (PA2)
- net +3V3: now also U4.5 (VOUT); no longer U4.4 (BYP)
- net +5V: no longer J1.5 (Pin_5)
- net 3V3_BYP: now also U4.4 (BYP); no longer U4.5 (VOUT)
- net GND: no longer J1.4 (Pin_4)
- net M1_SPD: no longer U1.17 (PB9)
- net M2_SPD: no longer U1.16 (PB8)
- no-connect marks 14 -> 13

Commit message: wip
Parts:
- added J10: Conn_01x06_Female, Connector_PinSocket_2.54mm:PinSocket_1x06_P2.54mm_Vertical, symbol Connector:Conn_01x06_Female
- added TP5, TP6: GND_TP, Connector_PinHeader_2.54mm:PinHeader_1x01_P2.54mm_Vertical, symbol Connector:TestPoint
Connections:
- net +5V: now also J10.5 (Pin_5)
- net GND: now also J10.4 (Pin_4), TP5.1, TP6.1
- net at C6.1, FB4.1, J1.2 (Pin_2): now also J10.2 (Pin_2)
- net at C8.1, FB3.2, J1.3 (Pin_3): now also J10.3 (Pin_3)
- no-connect marks 13 -> 17
Other:
- moved on the sheet: TP2
Changed lines of the file:
@@
 Wire Wire Line
 	3650 7200 3650 7575
-Wire Wire Line
-	3650 7575 3900 7575
 Connection ~ 3650 7575
 Wire Wire Line
@@
 L Connector:TestPoint TP2
 U 1 1 6391FDE6
-P 3900 7575
-F 0 "TP2" H 3958 7693 50  0000 L CNN
-F 1 "GND_TP" H 3958 7602 50  0000 L CNN
-F 2 "Connector_PinHeader_2.54mm:PinHeader_1x01_P2.54mm_Vertical" H 4100 7575 50  0001 C CNN
-F 3 "~" H 4100 7575 50  0001 C CNN
-	1    3900 7575
+P 3900 7500
+F 0 "TP2" H 3958 7618 50  0000 L CNN
+F 1 "GND_TP" H 3958 7527 50  0000 L CNN
+F 2 "Connector_PinHeader_2.54mm:PinHeader_1x01_P2.54mm_Vertical" H 4100 7500 50  0001 C CNN
+F 3 "~" H 4100 7500 50  0001 C CNN
+	1    3900 7500
 	1    0    0    -1
 $EndComp
@@
 	14425 7175 14575 7175
 Wire Wire Line
-	11725 7425 13450 7425
-Wire Wire Line
-	11725 7325 13850 7325
+	11725 7425 12800 7425
+Wire Wire Line
+	11725 7325 12625 7325
 Wire Wire Line
 	13850 7650 13850 7325
@@
 Connection ~ 8525 3975
 Connection ~ 8425 3975
+$Comp
+L Connector:TestPoint TP5
+U 1 1 647F84BA
+P 4275 7500
+F 0 "TP5" H 4333 7618 50  0000 L CNN
+F 1 "GND_TP" H 4333 7527 50  0000 L CNN
+F 2 "Connector_PinHeader_2.54mm:PinHeader_1x01_P2.54mm_Vertical" H 4475 7500 50  0001 C CNN
+F 3 "~" H 4475 7500 50  0001 C CNN
+	1    4275 7500
+	1    0    0    -1
+$EndComp
+$Comp
+L Connector:TestPoint TP6
+U 1 1 647F98B3
+P 4700 7500
+F 0 "TP6" H 4758 7618 50  0000 L CNN
+F 1 "GND_TP" H 4758 7527 50  0000 L CNN
+F 2 "Connector_PinHeader_2.54mm:PinHeader_1x01_P2.54mm_Vertical" H 4900 7500 50  0001 C CNN
+F 3 "~" H 4900 7500 50  0001 C CNN
+	1    4700 7500
+	1    0    0    -1
+$EndComp
+Wire Wire Line
+	4700 7575 4700 7500
+Wire Wire Line
+	3650 7575 3900 7575
+Wire Wire Line
+	4275 7500 4275 7575
+Connection ~ 4275 7575
+Wire Wire Line
+	4275 7575 4700 7575
+Wire Wire Line
+	3900 7500 3900 7575
+Connection ~ 3900 7575
+Wire Wire Line
+	3900 7575 4275 7575
+$Comp
+L Connector:Conn_01x06_Female J10
+U 1 1 64870CA0
+P 11475 8675
+F 0 "J10" H 11367 8150 50  0000 C CNN
+F 1 "Conn_01x06_Female" H 11367 8241 50  0000 C CNN
+F 2 "Connector_PinSocket_2.54mm:PinSocket_1x06_P2.54mm_Vertical" H 11475 8675 50  0001 C CNN
+F 3 "~" H 11475 8675 50  0001 C CNN
+	1    11475 8675
+	-1   0    0    1
+$EndComp
+Wire Wire Line
+	11675 8775 12800 8775
+Wire Wire Line
+	12800 8775 12800 7425
+Connection ~ 12800 7425
+Wire Wire Line
+	12800 7425 13450 7425
+Wire Wire Line
+	11675 8675 12625 8675
+Wire Wire Line
+	12625 8675 12625 7325
+Connection ~ 12625 7325
+Wire Wire Line
+	12625 7325 13850 7325
+Wire Wire Line
+	11675 8475 12225 8475
+Wire Wire Line
+	12225 8475 12225 8150
+Wire Wire Line
+	11675 8575 12225 8575
+Wire Wire Line
+	12225 8575 12225 9000
+$Comp
+L power:GND #PWR0118
+U 1 1 64919533
+P 12225 9000
+F 0 "#PWR0118" H 12225 8750 50  0001 C CNN
+F 1 "GND" H 12230 8827 50  0000 C CNN
+F 2 "" H 12225 9000 50  0001 C CNN
+F 3 "" H 12225 9000 50  0001 C CNN
+	1    12225 9000
+	1    0    0    -1
+$EndComp
+NoConn ~ 11675 8375
+NoConn ~ 11675 8875
+NoConn ~ 7650 3475
+NoConn ~ 7650 3575
+$Comp
+L power:+5V #PWR0117
+U 1 1 649E8DEB
+P 12225 8150
+F 0 "#PWR0117" H 12225 8000 50  0001 C CNN
+F 1 "+5V" H 12240 8323 50  0000 C CNN
+F 2 "" H 12225 8150 50  0001 C CNN
+F 3 "" H 12225 8150 50  0001 C CNN
+	1    12225 8150
+	1    0    0    -1
+$EndComp
 $EndSCHEMATC
