File: mouse_v2_PAIN.kicad_pcb (KiCad board)
At the start: 2 copper layers, 84.9 x 94.9 mm, 81 parts, among them J1 HC05 Header, J2 Serial Debug Header, J3 HC05_Key Jump, J4 Conn_ARM_JTAG_SWD_10, J5 SWD Header, M1 M1_Conn, M2 M2_Conn, Q0 Q_Photo_NPN, Q1 Q_Photo_NPN, Q2 Q_Photo_NPN, Q3 Q_Photo_NPN, Q4 Q_NMOS_SGD, Q5 Q_NMOS_SGD, Q6 Q_NMOS_SGD, Q7 Q_NMOS_SGD, Q8 Q_NMOS_SGD, SW1 SW, U1 YAAJ_BluePill_SWD_Breakout, U2 L293D, U3 LM1085-5.0

Commit message: a
Parts:
- added C11: 10uF, Capacitor_SMD:C_1206_3216Metric_Pad1.33x1.80mm_HandSolder, F.Cu at (250.0, 50.3)
- added C12: 0.1uF, Capacitor_SMD:C_1206_3216Metric_Pad1.33x1.80mm_HandSolder, F.Cu at (250.0, 53.6)
- added C13: 0.1uF, Capacitor_SMD:C_1206_3216Metric_Pad1.33x1.80mm_HandSolder, F.Cu at (403.9, 18.4)
- added C16: 100uF, Capacitor_THT:CP_Radial_D6.3mm_P2.50mm, F.Cu at (262.0, 50.3)
- added C17: 1uF, Capacitor_SMD:C_1206_3216Metric_Pad1.33x1.80mm_HandSolder, F.Cu at (167.8, 117.6)
- added C18: 1uF, Capacitor_SMD:C_1206_3216Metric_Pad1.33x1.80mm_HandSolder, F.Cu at (167.8, 121.0)
- added C19: 0.1uF, Capacitor_SMD:C_1206_3216Metric_Pad1.33x1.80mm_HandSolder, F.Cu at (393.4, 26.9)
- added M3: M1_Conn_Alt, Connector_PinHeader_2.54mm:PinHeader_1x06_P2.54mm_Vertical, F.Cu at (383.4, 19.0)
- added M4: M2_Conn_Alt, Connector_PinHeader_2.54mm:PinHeader_1x06_P2.54mm_Vertical, F.Cu at (388.1, 19.0)
- added R12: 47K, Resistor_SMD:R_1206_3216Metric_Pad1.30x1.75mm_HandSolder, F.Cu at (393.4, 30.2)
- added SW_RST1: SW, Button_Switch_THT:SW_PUSH_6mm, F.Cu at (392.4, 18.7)
- added TP3: TP_5V, Connector_PinHeader_2.54mm:PinHeader_1x01_P2.54mm_Vertical, F.Cu at (403.3, 22.4)
- added TP4: TP_3V3, Connector_PinHeader_2.54mm:PinHeader_1x01_P2.54mm_Vertical, F.Cu at (409.3, 19.0)
- added U4: APE8865Y5-33-HF-3, Package_TO_SOT_SMD:SOT-23-5, B.Cu at (173.5, 118.0)
- C1: value 100uF -> 0.1uF
- C10, C9: footprint Capacitor_SMD:C_1206_3216Metric_Pad1.42x1.75mm_HandSolder -> Capacitor_SMD:C_1206_3216Metric_Pad1.33x1.80mm_HandSolder
- JP1, JP3, R1, R10, R3, R5, R7, R9: moved to B.Cu
- M1, M2: footprint Connector_PinHeader_1.00mm:PinHeader_1x06_P1.00mm_Vertical -> Connector_JST:JST_SH_BM06B-SRSS-TB_1x06-1MP_P1.00mm_Vertical
- R11: value 10K -> 47K
- moved R10 137.9 mm to (136.2, 103.6), turned to 90 degrees
- moved JP1 127.4 mm to (131.8, 115.1)
- moved Q7 113.2 mm to (155.3, 134.1), turned to 180 degrees
- moved R9 109.9 mm to (138.6, 105.4), turned to 90 degrees
- moved Q5 102.1 mm to (161.0, 134.1), turned to 180 degrees
- moved J3 62.8 mm to (196.3, 154.9)
- moved JP3 55.7 mm to (131.8, 117.7), turned to 180 degrees
- moved R19 46.8 mm to (127.8, 60.3), turned to 270 degrees
- moved R21 43.7 mm to (124.9, 58.1), turned to 270 degrees
- moved R20 40.5 mm to (121.7, 58.4), turned to 270 degrees
- moved R5 38.7 mm to (200.8, 122.9), turned to 90 degrees
- moved C10 34.8 mm to (174.3, 65.3)
- moved M2 33.2 mm to (177.0, 74.7), turned to 180 degrees
- moved S2 29.4 mm to (176.9, 71.7)
- moved M1 28.5 mm to (143.0, 75.2), turned to 180 degrees
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Connections:
- D4 pad 1: GND -> LED_RED
- D5 pad 1: GND -> LED_GREEN
- D6 pad 1: GND -> LED_BLUE
- J4 pad 1: +3V3 -> 3V3_MCU
- J5 pad 1: +3V3 -> 3V3_MCU
- R19 pad 2: LED_RED -> +3V3
- R20 pad 2: LED_GREEN -> +3V3
- R21 pad 2: LED_BLUE -> +3V3
- U1 pad 20: +3V3 -> 3V3_MCU
- U1 pad 38: +3V3 -> 3V3_MCU
Other:
- board text added: "TODO isolate gnds in routing"
- board text removed: "Add motor mounts"
- board text removed: "GND"
- board text removed: "maybe power motor with regulator"

Commit message: started work on pcb
Parts:
- added JP4: Jumper_2_Open, Jumper:SolderJumper-2_P1.3mm_Bridged_Pad1.0x1.5mm, F.Cu at (208.4, 44.7)
- added JP5: Jumper_2_Open, Jumper:SolderJumper-2_P1.3mm_Bridged_Pad1.0x1.5mm, F.Cu at (207.0, 50.4)
- added L1: 10uH, Inductor_SMD:L_1206_3216Metric_Pad1.42x1.75mm_HandSolder, F.Cu at (149.9, 122.2)
- C1: footprint Capacitor_THT:CP_Radial_D6.3mm_P2.50mm -> Capacitor_SMD:C_1206_3216Metric_Pad1.33x1.80mm_HandSolder; moved to B.Cu
- C3, C4, C5, C6, C7, C8, C9, FB1, FB2, FB3, FB4, JP2, R13, R14, R22, R23: moved to B.Cu
- SW1, SW_RST1: footprint Button_Switch_THT:SW_PUSH_6mm -> Button_Switch_SMD:SW_SPST_REED_CT05-XXXX-G1
- moved TP4 282.3 mm to (154.1, 139.9)
- moved SW_RST1 281.4 mm to (137.4, 137.7), turned to 135 degrees
- moved C19 278.3 mm to (137.8, 137.2), turned to 270 degrees
- moved R12 272.3 mm to (142.0, 135.0), turned to 270 degrees
- moved M3 251.1 mm to (139.2, 77.5), turned to 90 degrees
- moved C13 239.8 mm to (168.5, 63.8), turned to 270 degrees
- moved M4 227.6 mm to (168.1, 77.6), turned to 90 degrees
- moved TP3 202.1 mm to (205.6, 64.5)
- moved FB1 145.3 mm to (146.5, 40.5), turned to 270 degrees
- moved JP2 144.6 mm to (120.8, 116.6)
- moved FB2 134.0 mm to (149.2, 39.2), turned to 90 degrees
- moved C5 133.5 mm to (146.3, 36.4), turned to 90 degrees
- moved C7 131.7 mm to (144.2, 38.8), turned to 90 degrees
- moved C12 125.6 mm to (144.4, 121.6)
- moved C11 118.6 mm to (152.3, 117.4)
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Connections:
- M1 pad 1: M2_OUT_1 -> GND
- M1 pad 2: M2_OUT_2 -> M2_ENC_B
- M1 pad 3: +3V3 -> M2_ENC_A
- M1 pad 4: M2_ENC_A -> +3V3
- M1 pad 5: M2_ENC_B -> M2_OUT_2
- M1 pad 6: GND -> M2_OUT_1
- M2 pad 1: M1_OUT_1 -> GND
- M2 pad 2: M1_OUT_2 -> M1_ENC_B
- M2 pad 3: +3V3 -> M1_ENC_A
- M2 pad 4: M1_ENC_A -> +3V3
- M2 pad 5: M1_ENC_B -> M1_OUT_2
- M2 pad 6: GND -> M1_OUT_1
- Q0 pad 1: +3V3 -> +3.3VA
- Q1 pad 1: +3V3 -> +3.3VA
- Q2 pad 1: +3V3 -> +3.3VA
- Q3 pad 1: +3V3 -> +3.3VA
- R1 pad 1: GND -> AGND
- R2 pad 1: GND -> AGND
- R3 pad 1: GND -> AGND
- R4 pad 1: GND -> AGND
- U1 pad 18: +5V -> Net-(U1-Pad18)
- U1 pad 20: 3V3_MCU -> +3V3
- U1 pad 38: 3V3_MCU -> +3V3
- U2 pad 12: GND -> MGND
- U2 pad 13: GND -> MGND
- U2 pad 4: GND -> MGND
- U2 pad 5: GND -> MGND
Routing:
- net +5V: track 0.00 -> 227.6 mm, vias 0 -> 6
- net +3V3: track 0.00 -> 55.0 mm
- net VCC: track 0.00 -> 50.4 mm, vias 0 -> 2
- net M1_OUT_1: track 0.00 -> 45.4 mm
- net M2_OUT_2: track 0.00 -> 39.8 mm
- net M2_OUT_1: track 0.00 -> 39.5 mm
- net M1_OUT_2: track 0.00 -> 38.2 mm
- net LED_RED: track 0.00 -> 32.2 mm, vias 0 -> 1
- net LED_BLUE: track 0.00 -> 31.6 mm, vias 0 -> 1
- net LED_GREEN: track 0.00 -> 29.7 mm, vias 0 -> 1
- net Net-(BT1-Pad1): track 0.00 -> 21.2 mm
- net GND: track 0.00 -> 16.2 mm
- net V_MOTOR: track 0.00 -> 13.3 mm
- net Net-(Q8-Pad3): track 0.00 -> 10.2 mm
- net Net-(D4-Pad2): track 0.00 -> 7.70 mm, vias 0 -> 1
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- removed copper zone on B.Cu, net /GND
- removed copper zone on F.Cu, net /GND
Other:
- board text added: "FIGURE OUT HOW TO GET THE GND VIAS"
- board text removed: "verify orientaiton"

Commit message: more tracing
Parts:
- C19, R12, R15, R16: moved to B.Cu
- R1, R2, R3, R4: moved to F.Cu
- moved TP4 47.9 mm to (110.1, 121.2)
- moved SW_RST1 42.9 mm to (180.3, 135.7), turned to 0 degrees
- moved C19 42.4 mm to (180.2, 135.8), turned to 0 degrees
- moved R12 37.1 mm to (177.7, 124.7), turned to 180 degrees
- moved C5 34.9 mm to (146.0, 71.2), turned to 270 degrees
- moved C7 33.2 mm to (151.0, 71.3), turned to 270 degrees
- moved FB2 32.1 mm to (147.7, 71.3), turned to 270 degrees
- moved FB1 31.0 mm to (149.4, 71.3), turned to 90 degrees
- moved R16 9.63 mm to (159.0, 134.7), turned to 270 degrees
- moved Q4 9.27 mm to (191.9, 122.3)
- moved R5 9.20 mm to (192.0, 120.0), turned to 180 degrees
- moved R13 8.32 mm to (188.0, 126.2)
- moved R15 7.44 mm to (133.7, 122.6)
- moved R8 7.00 mm to (154.4, 139.2)
- moved R1 6.82 mm to (188.0, 131.3)
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Connections:
- J4 pad 1: 3V3_MCU -> +3V3
- J5 pad 1: 3V3_MCU -> +3V3
- U1 pad 1: M1_FWD -> EMIT_1
- U1 pad 10: EMIT_3 -> LED_RED
- U1 pad 13: LED_RED -> EMIT_3
- U1 pad 14: M1_ENC_B -> M2_ENC_B
- U1 pad 15: M1_ENC_A -> M2_ENC_A
- U1 pad 16: M1_SPD -> M2_SPD
- U1 pad 17: M2_SPD -> M1_SPD
- U1 pad 2: M1_BACK -> M2_FWD
- U1 pad 29: RECEIV_1 -> RECEIV_2
- U1 pad 3: M2_FWD -> M1_BACK
- U1 pad 30: RECEIV_2 -> RECEIV_1
- U1 pad 31: M2_ENC_A -> M1_ENC_B
- U1 pad 32: M2_ENC_B -> M1_ENC_A
- U1 pad 35: LED_BLUE -> EMIT_4
- U1 pad 36: EMIT_4 -> EMIT_2
- U1 pad 5: BUTTON -> M1_FWD
- U1 pad 8: EMIT_2 -> BUTTON
- U1 pad 9: EMIT_1 -> LED_BLUE
Routing:
- net +5V: track 227.6 -> 400.0 mm
- net +3.3VA: track 0.00 -> 93.6 mm
- net AGND: track 0.00 -> 58.2 mm
- net RECEIV_2: track 0.00 -> 31.6 mm
- net SWDIO: track 5.73 -> 35.6 mm
- net USART1_RX: track 0.00 -> 28.7 mm
- net M2_BACK: track 0.00 -> 28.6 mm
- net BUTTON: track 2.87 -> 31.1 mm
- net RECEIV_4: track 0.00 -> 26.9 mm
- net USART1_TX: track 0.00 -> 26.7 mm
- net M2_FWD: track 0.00 -> 25.3 mm
- net SWDCLK: track 6.22 -> 31.5 mm, vias 0 -> 1
- net RECEIV_3: track 0.00 -> 24.5 mm, vias 0 -> 1
- net EMIT_4: track 0.00 -> 22.0 mm
- net USART2_TX: track 0.00 -> 21.8 mm
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Other:
- board text added: "Jonathan Low v0 2022"
- board text removed: "J. Low v0 2022"

Commit message: tracing
Parts:
- added J6: Conn_01x02_Female, Connector_PinSocket_2.00mm:PinSocket_1x02_P2.00mm_Vertical, F.Cu at (144.8, 135.3)
- added J7: Conn_01x02_Female, Connector_PinSocket_2.00mm:PinSocket_1x02_P2.00mm_Vertical, F.Cu at (135.1, 135.3)
- added J8: Conn_01x02_Female, Connector_PinSocket_2.00mm:PinSocket_1x02_P2.00mm_Vertical, F.Cu at (177.0, 138.5)
- added J9: Conn_01x02_Female, Connector_PinSocket_2.00mm:PinSocket_1x02_P2.00mm_Vertical, F.Cu at (184.7, 138.5)
- C11, C12, C17, C18, L1: moved to B.Cu
- moved C17 36.0 mm to (135.4, 101.7), turned to 270 degrees
- moved R17 33.8 mm to (145.8, 131.1), turned to 180 degrees
- moved C18 32.3 mm to (137.3, 110.3)
- moved R22 29.0 mm to (152.1, 118.8)
- moved R23 29.0 mm to (156.3, 118.9)
- moved U4 18.2 mm to (138.4, 101.3), turned to 270 degrees
- moved C11 17.7 mm to (137.3, 107.9)
- moved C12 17.6 mm to (137.3, 105.5)
- moved L1 16.8 mm to (140.6, 136.2), turned to 270 degrees
- moved BT_MH1 8.91 mm to (176.4, 100.6)
- moved J3 5.11 mm to (193.8, 105.5), turned to 0 degrees
- moved SW_RST1 1.08 mm to (180.8, 134.7)
- moved C19 1.08 mm to (180.7, 134.8)
Connections:
- U1 pad 10: LED_RED -> LED_GREEN
- U1 pad 12: LED_GREEN -> BUTTON
- U1 pad 31: M1_ENC_B -> M1_ENC_A
- U1 pad 32: M1_ENC_A -> M1_ENC_B
- U1 pad 8: BUTTON -> LED_RED
Routing:
- net +3V3: track 66.8 -> 188.6 mm, vias 0 -> 1
- net M1_ENC_A: track 6.22 -> 91.7 mm
- net M1_ENC_B: track 6.85 -> 88.8 mm
- net M2_FWD: track 25.3 -> 96.3 mm
- net M1_BACK: track 13.7 -> 83.6 mm
- net LED_RED: track 32.2 -> 97.7 mm, vias 1 -> 2
- net LED_BLUE: track 31.6 -> 94.2 mm, vias 1 -> 2
- net M2_BACK: track 28.6 -> 88.8 mm
- net M1_FWD: track 19.1 -> 78.4 mm
- net LED_GREEN: track 29.7 -> 88.6 mm, vias 1 -> 2
- net BUZZER: track 18.6 -> 77.2 mm, vias 0 -> 1
- net USART2_RX: track 20.9 -> 72.8 mm, vias 0 -> 1
- net BUTTON: track 31.1 -> 81.6 mm
- net USART2_TX: track 21.8 -> 72.0 mm, vias 0 -> 1
- net M2_SPD: track 20.3 -> 60.1 mm, vias 0 -> 1
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
Commit message: tracing
Parts:
- removed JP5: Jumper_2_Open, Jumper:SolderJumper-2_P1.3mm_Bridged_Pad1.0x1.5mm
- added C14: 1uF, Capacitor_SMD:C_1206_3216Metric_Pad1.33x1.80mm_HandSolder, B.Cu at (145.0, 138.0)
- added C15: 1uF, Capacitor_SMD:C_1206_3216Metric_Pad1.33x1.80mm_HandSolder, B.Cu at (188.3, 135.3)
- added C20: 1uF, Capacitor_SMD:C_1206_3216Metric_Pad1.33x1.80mm_HandSolder, B.Cu at (132.3, 134.0)
- added C21: 1uF, Capacitor_SMD:C_1206_3216Metric_Pad1.33x1.80mm_HandSolder, B.Cu at (173.3, 137.7)
- moved JP4 101.2 mm to (158.9, 133.0), turned to 90 degrees
- moved TP3 45.7 mm to (160.1, 60.3)
- moved TP2 40.5 mm to (156.8, 57.0), turned to 180 degrees
- moved TP1 26.1 mm to (192.7, 56.6)
- moved TP4 19.6 mm to (121.0, 104.9), turned to 90 degrees
- moved R22 5.84 mm to (157.7, 120.4)
- moved C2 5.04 mm to (192.0, 61.9), turned to 180 degrees
- moved C9 2.86 mm to (191.0, 68.0)
- moved C1 2.70 mm to (193.4, 68.0)
- moved R23 2.05 mm to (154.9, 120.4), turned to 90 degrees
Connections:
- C2 pad 1: GND -> VCC
- C2 pad 2: VCC -> GND
- U2 pad 12: MGND -> GND
- U2 pad 13: MGND -> GND
- U2 pad 4: MGND -> GND
- U2 pad 5: MGND -> GND
Routing:
- net VCC: track 50.4 -> 114.9 mm, vias 2 -> 4
- net RST: track 15.9 -> 68.9 mm, vias 0 -> 3
- net AGND: track 79.0 -> 94.3 mm, vias 0 -> 4
- net MGND: track 12.7 -> 0.00 mm
- net GND: track 3.21 -> 15.9 mm, vias 0 -> 80
- net +3.3VA: track 98.9 -> 110.2 mm
- net V_METER: track 5.37 -> 13.6 mm
- net +3V3: track 188.6 -> 195.5 mm
- net Net-(S1-Pad3): track 0.00 -> 6.18 mm
- net +5V: track 419.2 -> 424.1 mm
- net HC05_Key: track 3.99 -> 6.13 mm
- net M1_BACK: track 83.6 -> 81.8 mm
- net EMIT_3: track 36.5 -> 38.2 mm
- net M2_FWD: track 96.3 -> 95.8 mm
- net (no net): vias 0 -> 1
- added copper zone on B.Cu, net GND
- added copper zone on F.Cu, net GND

Commit message: tracing
Parts:
- added Q10: Q_NMOS_GSD, Package_TO_SOT_SMD:SOT-23, F.Cu at (169.7, 135.5)
- added Q11: Q_NMOS_GSD, Package_TO_SOT_SMD:SOT-23, F.Cu at (134.2, 122.2)
- added Q12: Q_NMOS_GSD, Package_TO_SOT_SMD:SOT-23, F.Cu at (153.5, 138.9)
- added Q9: Q_NMOS_GSD, Package_TO_SOT_SMD:SOT-23, F.Cu at (191.5, 118.6)
- U3: footprint Package_TO_SOT_SMD:TO-263-3_TabPin2 -> custom:VREG_TO-263-3_TabPin2
- moved BT_MH2 52.9 mm to (151.8, 100.3)
- moved BT_MH1 10.1 mm to (166.3, 100.3)
Routing:
- net +3V3: track 195.5 -> 257.0 mm, vias 1 -> 4
- net Net-(Q10-Pad3): track 4.09 -> 10.8 mm
- net EMIT_2: track 19.2 -> 24.8 mm
- net Net-(Q11-Pad3): track 2.68 -> 7.90 mm, vias 0 -> 1
- net GND: track 15.9 -> 19.1 mm, vias 80 -> 182
- net EMIT_1: track 16.3 -> 19.3 mm
- net Net-(Q4-Pad3): track 3.04 -> 5.82 mm, vias 0 -> 1
- net Net-(Q12-Pad3): track 3.83 -> 6.37 mm, vias 0 -> 1
- net EMIT_4: track 22.0 -> 24.3 mm
- net EMIT_3: track 38.2 -> 39.5 mm
- net RST: track 68.9 -> 69.2 mm, vias 3 -> 4
Other:
- board text removed: "FIGURE OUT HOW TO GET THE GND VIAS"
- board text removed: "TODO isolate gnds in routing"

Commit message: label cleanup
Other:
- board text added: "SOT PIN OUT OFF"
- board text added: "d"
- board text added: "g"
- board text added: "s"

Commit message: v0 PCB
Parts:
- added C25: 10nF, Capacitor_SMD:C_1206_3216Metric_Pad1.33x1.80mm_HandSolder, F.Cu at (138.0, 97.6)
- moved BT_MH1 1.88 mm to (168.2, 100.3)
Connections:
- U4 pad 4: Net-(U4-Pad4) -> +3V3
- U4 pad 5: +3V3 -> 3V3_BYP
Routing:
- net 3V3_BYP: track 0.00 -> 3.46 mm, vias 0 -> 1
- net +3V3: track 257.0 -> 257.8 mm
- net +5V: track 424.1 -> 423.3 mm
Other:
- board text added: "3V3"
- board text added: "GND"
- board text added: "RST"
- board text added: "SWDCLK"
- board text added: "SWDIO"
- board text removed: "SOT PIN OUT OFF"
