File: mouse_v2_PAIN.kicad_pcb (KiCad board)
At the start: 2 copper layers, 84.9 x 94.9 mm, 110 parts, among them J1 HC05 Header, J2 Serial Debug Header, J3 HC05_Key Jump, J4 Conn_ARM_JTAG_SWD_10, J5 SWD Header, J6 Conn_01x02_Female, J7 Conn_01x02_Female, J8 Conn_01x02_Female, J9 Conn_01x02_Female, M1 M1_Conn, M2 M2_Conn, M3 M1_Conn_Alt, M4 M2_Conn_Alt, Q0 Q_Photo_NPN, Q1 Q_Photo_NPN, Q10 Q_NMOS_GSD, Q11 Q_NMOS_GSD, Q12 Q_NMOS_GSD, Q2 Q_Photo_NPN, Q3 Q_Photo_NPN, Q4 Q_NMOS_SGD, Q5 Q_NMOS_SGD, Q6 Q_NMOS_SGD, Q7 Q_NMOS_SGD, Q8 Q_NMOS_SGD, Q9 Q_NMOS_GSD, SW1 SW, U1 YAAJ_BluePill_SWD_Breakout, U2 L293D, U3 LM1085-5.0, U4 APE8865Y5-33-HF-3

Commit message: changes for v0.1 wip
Parts:
- removed C5, C7: 22pF, Capacitor_SMD:C_0603_1608Metric_Pad1.08x0.95mm_HandSolder
- removed FB1, FB2: HZ0603C601R-10, Resistor_SMD:R_0603_1608Metric_Pad0.98x0.95mm_HandSolder
- removed J2: Serial Debug Header, Connector_PinHeader_2.54mm:PinHeader_1x06_P2.54mm_Vertical
- removed J3: HC05_Key Jump, Connector_PinHeader_2.54mm:PinHeader_1x02_P2.54mm_Vertical
- J1: value HC05 Header -> Serial Debug Header
Connections:
- J1 pad 4: GND -> Net-(J1-Pad4)
- J1 pad 5: +5V -> Net-(J1-Pad5)
- J1 pad 6: HC05_Key -> GND
- U1 pad 16: M2_SPD -> Net-(U1-Pad16)
- U1 pad 17: M1_SPD -> Net-(U1-Pad17)
- U1 pad 27: USART2_TX -> M2_SPD
- U1 pad 28: USART2_RX -> M1_SPD
- U1 pad 41: (no net) -> GND
- U1 pad 42: SWDIO -> SWDCLK
- U1 pad 43: SWDCLK -> SWDIO
- U1 pad 44: GND -> (no net)
- U4 pad 4: +3V3 -> 3V3_BYP
- U4 pad 5: 3V3_BYP -> +3V3
Routing:
- net USART2_RX: track 72.8 -> 0.00 mm, vias 1 -> 0
- net USART2_TX: track 72.0 -> 0.00 mm, vias 1 -> 0
- net M2_SPD: track 60.1 -> 78.7 mm
- net M1_SPD: track 49.3 -> 67.0 mm, vias 1 -> 2
- net Net-(C5-Pad1): track 16.0 -> 0.00 mm
- net Net-(C7-Pad1): track 15.6 -> 0.00 mm
- net HC05_Key: track 6.13 -> 0.00 mm
- net SWDIO: track 32.7 -> 27.7 mm
- net +5V: track 423.3 -> 421.1 mm
- net SWDCLK: track 29.8 -> 30.8 mm
- net 3V3_BYP: track 3.46 -> 4.44 mm
- net +3V3: track 257.8 -> 257.1 mm

Commit message: wip
Parts:
- removed JP2: JP_GND, Jumper:SolderJumper-2_P1.3mm_Open_Pad1.0x1.5mm
- added J10: Conn_01x06_Female, Connector_PinSocket_2.54mm:PinSocket_1x06_P2.54mm_Vertical, F.Cu at (200.3, 117.8)
- added JP_GND: JP_GND, Jumper:SolderJumper-2_P1.3mm_Open_Pad1.0x1.5mm, B.Cu at (123.8, 108.9)
- added TP5: GND_TP, Connector_PinHeader_2.54mm:PinHeader_1x01_P2.54mm_Vertical, F.Cu at (144.4, 56.3)
- added TP6: GND_TP, Connector_PinHeader_2.54mm:PinHeader_1x01_P2.54mm_Vertical, F.Cu at (140.8, 56.2)
- C6, C8, FB3, FB4: moved to F.Cu
- moved TP2 83.8 mm to (136.7, 138.3)
- moved TP3 8.35 mm to (152.2, 57.6)
- moved J4 4.96 mm to (121.1, 114.0), turned to 180 degrees
- moved C6 3.75 mm to (193.1, 116.1)
- moved FB4 3.72 mm to (193.1, 114.5)
- moved C8 3.64 mm to (193.1, 111.1)
- moved FB3 3.64 mm to (193.1, 112.7)
- moved J1 3.23 mm to (196.6, 117.8)
- moved JP_RST 0.52 mm to (124.0, 115.6)
- renumbered JP3 to JP_RST, JP1 to JP_SWO
Routing:
- net +5V: track 421.1 -> 448.1 mm
- net SWDCLK: track 30.8 -> 45.8 mm, vias 0 -> 1
- net Net-(J4-Pad10): track 2.33 -> 14.6 mm, vias 0 -> 2
- net Net-(J4-Pad6): track 2.02 -> 14.1 mm, vias 0 -> 2
- net SWDIO: track 27.7 -> 38.2 mm, vias 0 -> 1
- net Net-(C6-Pad1): track 3.85 -> 8.16 mm
- net +3V3: track 257.1 -> 261.2 mm
- net Net-(C8-Pad1): track 3.86 -> 7.91 mm
- net USART1_RX: track 28.3 -> 24.6 mm, vias 1 -> 0
- net USART1_TX: track 25.5 -> 21.8 mm, vias 1 -> 0
- net M1_OUT_1: track 45.4 -> 44.1 mm
- net V_MOTOR: track 13.6 -> 12.6 mm
- net Net-(J4-Pad9): track 2.80 -> 2.12 mm
- net GND: vias 182 -> 175
Other:
- board text added: "Jonathan Low v0.1 2022"
- board text removed: "Jonathan Low v0 2022"

Commit message: minor
Parts:
- moved J1 3.84 mm to (200.5, 117.8)
- moved J10 3.43 mm to (196.8, 117.8)
Routing:
- net +5V: track 448.1 -> 452.7 mm
- net GND: vias 175 -> 180
Other:
- board text added: "5V"
- board text added: "HC05"
- board text added: "Jonathan Low v0.1 2023"
- board text added: "RX"
- board text added: "Serial Debug"
- board text added: "TX"
- board text removed: "Jonathan Low v0.1 2022"
